File: LT3060board_out.sch (KiCad schematic (older format))
At the start: 6 parts, among them IC1 LT3060-TSOT, K1 CONN_3

Commit message: Version with 3 TVS-diodes for protection.
Parts:
- added D1, D2, D3: TVS, symbol TVS
Connections:
- wire segments 26 -> 37
Changed lines of the file:
@@
 Sheet 1 1
 Title ""
-Date "2 aug 2014"
+Date "27 aug 2014"
 Rev ""
 Comp ""
@@
 $EndComp
 $Comp
-L GND #PWR2
+L GND #PWR01
 U 1 1 53DBB588
 P 4600 3600
-F 0 "#PWR2" H 4600 3600 30  0001 C CNN
+F 0 "#PWR01" H 4600 3600 30  0001 C CNN
 F 1 "GND" H 4600 3530 30  0001 C CNN
 F 2 "" H 4600 3600 60  0000 C CNN
@@
 	4600 4100 4600 4000
 Wire Wire Line
-	4600 4000 6150 4000
-Wire Wire Line
-	6150 4000 6150 2500
-Wire Wire Line
-	6150 2500 5300 2500
+	4600 4000 6500 4000
+Wire Wire Line
+	6500 4000 6500 2500
+Wire Wire Line
+	6500 2500 5300 2500
 $Comp
 L C C2
@@
 $EndComp
 $Comp
-L GND #PWR3
+L GND #PWR02
 U 1 1 53DBB632
 P 4800 3900
-F 0 "#PWR3" H 4800 3900 30  0001 C CNN
+F 0 "#PWR02" H 4800 3900 30  0001 C CNN
 F 1 "GND" H 4800 3830 30  0001 C CNN
 F 2 "" H 4800 3900 60  0000 C CNN
@@
 $EndComp
 $Comp
-L GND #PWR4
+L GND #PWR03
 U 1 1 53DBB65C
 P 5850 3000
-F 0 "#PWR4" H 5850 3000 30  0001 C CNN
+F 0 "#PWR03" H 5850 3000 30  0001 C CNN
 F 1 "GND" H 5850 2930 30  0001 C CNN
 F 2 "" H 5850 3000 60  0000 C CNN
@@
 $EndComp
 $Comp
-L GND #PWR1
+L GND #PWR04
 U 1 1 53DBB662
 P 3550 3200
-F 0 "#PWR1" H 3550 3200 30  0001 C CNN
+F 0 "#PWR04" H 3550 3200 30  0001 C CNN
 F 1 "GND" H 3550 3130 30  0001 C CNN
 F 2 "" H 3550 3200 60  0000 C CNN
@@
 	4800 3850 4800 3900
 $Comp
-L PWR_FLAG #FLG3
+L PWR_FLAG #FLG05
 U 1 1 53DBCC7F
 P 5850 2450
-F 0 "#FLG3" H 5850 2545 30  0001 C CNN
+F 0 "#FLG05" H 5850 2545 30  0001 C CNN
 F 1 "PWR_FLAG" H 5850 2630 30  0000 C CNN
 F 2 "" H 5850 2450 60  0000 C CNN
@@
 $EndComp
 $Comp
-L PWR_FLAG #FLG1
+L PWR_FLAG #FLG06
 U 1 1 53DBCC8C
 P 3750 2450
-F 0 "#FLG1" H 3750 2545 30  0001 C CNN
+F 0 "#FLG06" H 3750 2545 30  0001 C CNN
 F 1 "PWR_FLAG" H 3750 2630 30  0000 C CNN
 F 2 "" H 3750 2450 60  0000 C CNN
@@
 $EndComp
 $Comp
-L PWR_FLAG #FLG2
+L PWR_FLAG #FLG07
 U 1 1 53DBCC92
 P 4200 3600
-F 0 "#FLG2" H 4200 3695 30  0001 C CNN
+F 0 "#FLG07" H 4200 3695 30  0001 C CNN
 F 1 "PWR_FLAG" H 4200 3780 30  0000 C CNN
 F 2 "" H 4200 3600 60  0000 C CNN
@@
 	4200 3600 4200 3650
 Wire Wire Line
-	4200 3650 4500 3650
+	3900 3650 4500 3650
 Connection ~ 4500 3650
 Text Label 3550 2500 0    60   ~ 0
@@
 	1    0    0    -1
 $EndComp
+$Comp
+L TVS D2
+U 1 1 53FE1CF8
+P 4550 1950
+F 0 "D2" H 4500 2050 50  0000 C CNN
+F 1 "TVS" H 4500 1850 40  0000 C CNN
+F 2 "" H 4650 1950 60  0000 C CNN
+F 3 "http://www.littelfuse.com/~/media/electronics/datasheets/tvs_diodes/littelfuse_tvs_diode_smdj_datasheet.pdf.pdf" H 4650 1950 60 0001 C CNN ""
+F 4 "33" H 4550 1950 60  0001 C CNN "Breakdown Voltage"
+F 5 "1" H 4550 1950 60  0001 C CNN "Bidirectional Channels"
+F 6 "-" H 4550 1950 60  0001 C CNN "Unidirectional Channels"
+F 7 "SMDJ30CACT-ND" H 4550 1950 60 0001 C CNN "Digi-Key Part Number"
+F 8 "SMDJ30CA" H 4550 1950 60 0001 C CNN "Manufacturer Part Number"
+F 9 "1.290000e+000" H 4550 1950 60 0001 C CNN "Price"
+	1    4550 1950
+	1    0    0    -1
+$EndComp
+Wire Wire Line
+	3850 2500 3850 2350
+Wire Wire Line
+	3850 2350 4000 2350
+Wire Wire Line
+	4000 2350 4000 1950
+Wire Wire Line
+	4000 1950 4300 1950
+Connection ~ 3850 2500
+Wire Wire Line
+	4800 1950 5350 1950
+Wire Wire Line
+	5350 1950 5350 2500
+Connection ~ 5350 2500
+$Comp
+L TVS D1
+U 1 1 53FE1D92
+P 3900 3250
+F 0 "D1" H 3850 3350 50  0000 C CNN
+F 1 "TVS" H 3850 3150 40  0000 C CNN
+F 2 "" H 4000 3250 60  0000 C CNN
+F 3 "http://www.littelfuse.com/~/media/electronics/datasheets/tvs_diodes/littelfuse_tvs_diode_smdj_datasheet.pdf.pdf" H 4000 3250 60 0001 C CNN ""
+F 4 "33" H 3900 3250 60  0001 C CNN "Breakdown Voltage"
+F 5 "1" H 3900 3250 60  0001 C CNN "Bidirectional Channels"
+F 6 "-" H 3900 3250 60  0001 C CNN "Unidirectional Channels"
+F 7 "SMDJ30CACT-ND" H 3900 3250 60 0001 C CNN "Digi-Key Part Number"
+F 8 "SMDJ30CA" H 3900 3250 60 0001 C CNN "Manufacturer Part Number"
+F 9 "1.290000e+000" H 3900 3250 60 0001 C CNN "Price"
+	1    3900 3250
+	0    -1   -1   0
+$EndComp
+Wire Wire Line
+	3900 3000 3750 3000
+Connection ~ 3750 3000
+Wire Wire Line
+	3900 3500 3900 3650
+Connection ~ 4200 3650
+$Comp
+L TVS D3
+U 1 1 53FE1E08
+P 6250 2800
+F 0 "D3" H 6200 2900 50  0000 C CNN
+F 1 "TVS" H 6200 2700 40  0000 C CNN
+F 2 "" H 6350 2800 60  0000 C CNN
+F 3 "http://www.littelfuse.com/~/media/electronics/datasheets/tvs_diodes/littelfuse_tvs_diode_smdj_datasheet.pdf.pdf" H 6350 2800 60 0001 C CNN ""
+F 4 "33" H 6250 2800 60  0001 C CNN "Breakdown Voltage"
+F 5 "1" H 6250 2800 60  0001 C CNN "Bidirectional Channels"
+F 6 "-" H 6250 2800 60  0001 C CNN "Unidirectional Channels"
+F 7 "SMDJ30CACT-ND" H 6250 2800 60 0001 C CNN "Digi-Key Part Number"
+F 8 "SMDJ30CA" H 6250 2800 60 0001 C CNN "Manufacturer Part Number"
+F 9 "1.290000e+000" H 6250 2800 60 0001 C CNN "Price"
+	1    6250 2800
+	0    -1   -1   0
+$EndComp
+Wire Wire Line
+	6250 2550 6250 2500
+Wire Wire Line
+	6250 2500 6300 2500
+Connection ~ 6300 2500
+$Comp
+L GND #PWR08
+U 1 1 53FE1E4A
+P 6250 3150
+F 0 "#PWR08" H 6250 3150 30  0001 C CNN
+F 1 "GND" H 6250 3080 30  0001 C CNN
+F 2 "" H 6250 3150 60  0000 C CNN
+F 3 "" H 6250 3150 60  0000 C CNN
+	1    6250 3150
+	1    0    0    -1
+$EndComp
+Wire Wire Line
+	6250 3050 6250 3150
 $EndSCHEMATC

Commit message: LT3060 protected by more compact TVS-diodes
Parts:
- removed D1, D2, D3: TVS, symbol TVS
- added D1, D2: TVS, ~, symbol TVSCOMA
Changed lines of the file:
@@
 Wire Wire Line
 	6500 4000 6500 2500
-Wire Wire Line
-	6500 2500 5300 2500
 $Comp
 L C C2
@@
 Wire Wire Line
 	4200 3600 4200 3650
-Wire Wire Line
-	3900 3650 4500 3650
 Connection ~ 4500 3650
 Text Label 3550 2500 0    60   ~ 0
@@
 	1    0    0    -1
 $EndComp
-$Comp
-L TVS D2
-U 1 1 53FE1CF8
-P 4550 1950
-F 0 "D2" H 4500 2050 50  0000 C CNN
-F 1 "TVS" H 4500 1850 40  0000 C CNN
-F 2 "" H 4650 1950 60  0000 C CNN
-F 3 "http://www.littelfuse.com/~/media/electronics/datasheets/tvs_diodes/littelfuse_tvs_diode_smdj_datasheet.pdf.pdf" H 4650 1950 60 0001 C CNN ""
-F 4 "33" H 4550 1950 60  0001 C CNN "Breakdown Voltage"
-F 5 "1" H 4550 1950 60  0001 C CNN "Bidirectional Channels"
-F 6 "-" H 4550 1950 60  0001 C CNN "Unidirectional Channels"
-F 7 "SMDJ30CACT-ND" H 4550 1950 60 0001 C CNN "Digi-Key Part Number"
-F 8 "SMDJ30CA" H 4550 1950 60 0001 C CNN "Manufacturer Part Number"
-F 9 "1.290000e+000" H 4550 1950 60 0001 C CNN "Price"
-	1    4550 1950
-	1    0    0    -1
-$EndComp
 Wire Wire Line
 	3850 2500 3850 2350
@@
 	3850 2350 4000 2350
 Wire Wire Line
-	4000 2350 4000 1950
-Wire Wire Line
-	4000 1950 4300 1950
+	4000 2350 4000 1800
+Wire Wire Line
+	4000 1800 4350 1800
 Connection ~ 3850 2500
 Wire Wire Line
-	4800 1950 5350 1950
-Wire Wire Line
-	5350 1950 5350 2500
+	5350 1800 5350 2500
 Connection ~ 5350 2500
-$Comp
-L TVS D1
-U 1 1 53FE1D92
-P 3900 3250
-F 0 "D1" H 3850 3350 50  0000 C CNN
-F 1 "TVS" H 3850 3150 40  0000 C CNN
-F 2 "" H 4000 3250 60  0000 C CNN
-F 3 "http://www.littelfuse.com/~/media/electronics/datasheets/tvs_diodes/littelfuse_tvs_diode_smdj_datasheet.pdf.pdf" H 4000 3250 60 0001 C CNN ""
-F 4 "33" H 3900 3250 60  0001 C CNN "Breakdown Voltage"
-F 5 "1" H 3900 3250 60  0001 C CNN "Bidirectional Channels"
-F 6 "-" H 3900 3250 60  0001 C CNN "Unidirectional Channels"
-F 7 "SMDJ30CACT-ND" H 3900 3250 60 0001 C CNN "Digi-Key Part Number"
-F 8 "SMDJ30CA" H 3900 3250 60 0001 C CNN "Manufacturer Part Number"
-F 9 "1.290000e+000" H 3900 3250 60 0001 C CNN "Price"
-	1    3900 3250
-	0    -1   -1   0
-$EndComp
-Wire Wire Line
-	3900 3000 3750 3000
-Connection ~ 3750 3000
-Wire Wire Line
-	3900 3500 3900 3650
-Connection ~ 4200 3650
-$Comp
-L TVS D3
-U 1 1 53FE1E08
-P 6250 2800
-F 0 "D3" H 6200 2900 50  0000 C CNN
-F 1 "TVS" H 6200 2700 40  0000 C CNN
-F 2 "" H 6350 2800 60  0000 C CNN
-F 3 "http://www.littelfuse.com/~/media/electronics/datasheets/tvs_diodes/littelfuse_tvs_diode_smdj_datasheet.pdf.pdf" H 6350 2800 60 0001 C CNN ""
-F 4 "33" H 6250 2800 60  0001 C CNN "Breakdown Voltage"
-F 5 "1" H 6250 2800 60  0001 C CNN "Bidirectional Channels"
-F 6 "-" H 6250 2800 60  0001 C CNN "Unidirectional Channels"
-F 7 "SMDJ30CACT-ND" H 6250 2800 60 0001 C CNN "Digi-Key Part Number"
-F 8 "SMDJ30CA" H 6250 2800 60 0001 C CNN "Manufacturer Part Number"
-F 9 "1.290000e+000" H 6250 2800 60 0001 C CNN "Price"
-	1    6250 2800
-	0    -1   -1   0
-$EndComp
-Wire Wire Line
-	6250 2550 6250 2500
-Wire Wire Line
-	6250 2500 6300 2500
-Connection ~ 6300 2500
 $Comp
 L GND #PWR08
 U 1 1 53FE1E4A
-P 6250 3150
-F 0 "#PWR08" H 6250 3150 30  0001 C CNN
-F 1 "GND" H 6250 3080 30  0001 C CNN
-F 2 "" H 6250 3150 60  0000 C CNN
-F 3 "" H 6250 3150 60  0000 C CNN
-	1    6250 3150
-	1    0    0    -1
-$EndComp
-Wire Wire Line
-	6250 3050 6250 3150
+P 4250 2200
+F 0 "#PWR08" H 4250 2200 30  0001 C CNN
+F 1 "GND" H 4250 2130 30  0001 C CNN
+F 2 "" H 4250 2200 60  0000 C CNN
+F 3 "" H 4250 2200 60  0000 C CNN
+	1    4250 2200
+	1    0    0    -1
+$EndComp
+$Comp
+L TVSCOMA D1
+U 1 1 53FE53A3
+P 4650 1800
+F 0 "D1" H 4650 1900 50  0000 C CNN
+F 1 "TVS" H 4800 1700 40  0000 C CNN
+F 2 "~" H 4750 1800 60  0000 C CNN
+F 3 "http://www.littelfuse.com/~/media/electronics/datasheets/tvs_diode_arrays/littelfuse_tvs_diode_array_sm_datasheet.pdf.pdf" H 4750 1800 60 0001 C CNN ""
+F 4 "36" H 4650 1800 60  0001 C CNN "Reverse Standoff Voltage"
+F 5 "-" H 4650 1800 60  0001 C CNN "Bidirectional Channels"
+F 6 "2" H 4650 1800 60  0001 C CNN "Unidirectional Channels"
+F 7 "F6350CT-ND" H 4650 1800 60 0001 C CNN "Digi-Key Part Number"
+F 8 "SM36-02HTG" H 4650 1800 60 0001 C CNN "Manufacturer Part Number"
+F 9 "5.900000e-001" H 4650 1800 60 0001 C CNN "Price"
+	1    4650 1800
+	1    0    0    -1
+$EndComp
+Wire Wire Line
+	6500 2500 5300 2500
+$Comp
+L TVSCOMA D2
+U 1 1 53FE54F9
+P 4650 2150
+F 0 "D2" H 4650 2250 50  0000 C CNN
+F 1 "TVS" H 4800 2050 40  0000 C CNN
+F 2 "~" H 4750 2150 60  0000 C CNN
+F 3 "http://www.littelfuse.com/~/media/electronics/datasheets/tvs_diode_arrays/littelfuse_tvs_diode_array_sm_datasheet.pdf.pdf" H 4750 2150 60 0001 C CNN ""
+F 4 "36" H 4650 2150 60  0001 C CNN "Reverse Standoff Voltage"
+F 5 "-" H 4650 2150 60  0001 C CNN "Bidirectional Channels"
+F 6 "2" H 4650 2150 60  0001 C CNN "Unidirectional Channels"
+F 7 "F6350CT-ND" H 4650 2150 60 0001 C CNN "Digi-Key Part Number"
+F 8 "SM36-02HTG" H 4650 2150 60 0001 C CNN "Manufacturer Part Number"
+F 9 "5.900000e-001" H 4650 2150 60 0001 C CNN "Price"
+	1    4650 2150
+	-1   0    0    1
+$EndComp
+Wire Wire Line
+	4650 2000 4650 1950
+Wire Wire Line
+	4950 1800 5350 1800
+Wire Wire Line
+	4350 2150 4250 2150
+Wire Wire Line
+	4250 2150 4250 2200
+$Comp
+L GND #PWR09
+U 1 1 53FE55ED
+P 5050 2200
+F 0 "#PWR09" H 5050 2200 30  0001 C CNN
+F 1 "GND" H 5050 2130 30  0001 C CNN
+F 2 "" H 5050 2200 60  0000 C CNN
+F 3 "" H 5050 2200 60  0000 C CNN
+	1    5050 2200
+	1    0    0    -1
+$EndComp
+Wire Wire Line
+	5050 2200 5050 2150
+Wire Wire Line
+	5050 2150 4950 2150
+Wire Wire Line
+	4200 3650 4500 3650
 $EndSCHEMATC

Commit message: test useable (z-diode test, cap test, voltage test) - no over current test
Parts:
- C1, C4: Tolerance 30% -> 21%
- C2, C3: Digi-Key Part Number 1276-2119-1-ND -> 1276-1009-1-ND; Manufacturer Part Number CL10B822KB8NNNC -> CL10B103KB8NNNC; Tolerance 30% -> 21%
- D1, D2: value TVS -> TVScomA
Changed lines of the file:
@@
 EESchema Schematic File Version 2
 LIBS:power
-LIBS:device
 LIBS:transistors
 LIBS:conn
@@
 LIBS:contrib
 LIBS:valves
+LIBS:device
 LIBS:LT3060board-cache
 EELAYER 27 0
@@
 Sheet 1 1
 Title ""
-Date "27 aug 2014"
+Date "24 may 2015"
 Rev ""
 Comp ""
@@
 F 1 "10nF" H 4806 3565 40  0000 L CNN
 F 2 "0603" H 4838 3500 30  0000 C CNN
-F 3 "http://www.samsungsem.com/servlet/FileDownload?type=spec&file=CL10B822KB8NNNC.pdf" H 4800 3650 60 0001 C CNN ""
+F 3 "http://www.samsungsem.com/servlet/FileDownload?type=spec&file=CL10B103KB8NNNC.pdf" H 4800 3650 60 0001 C CNN ""
 F 4 "50V" H 4800 3650 60  0001 C CNN "Voltage"
-F 5 "30%" H 4800 3650 60  0001 C CNN "Tolerance"
-F 6 "1276-2119-1-ND" H 4800 3650 60 0001 C CNN "Digi-Key Part Number"
-F 7 "CL10B822KB8NNNC" H 4800 3650 60 0001 C CNN "Manufacturer Part Number"
+F 5 "21%" H 4800 3650 60  0001 C CNN "Tolerance"
+F 6 "1276-1009-1-ND" H 4800 3650 60 0001 C CNN "Digi-Key Part Number"
+F 7 "CL10B103KB8NNNC" H 4800 3650 60 0001 C CNN "Manufacturer Part Number"
 F 8 "1.000000e-001" H 4800 3650 60 0001 C CNN "Price"
 	1    4800 3650
@@
 F 1 "10nF" H 5556 2665 40  0000 L CNN
 F 2 "0603" H 5588 2600 30  0000 C CNN
-F 3 "http://www.samsungsem.com/servlet/FileDownload?type=spec&file=CL10B822KB8NNNC.pdf" H 5550 2750 60 0001 C CNN ""
+F 3 "http://www.samsungsem.com/servlet/FileDownload?type=spec&file=CL10B103KB8NNNC.pdf" H 5550 2750 60 0001 C CNN ""
 F 4 "50V" H 5550 2750 60  0001 C CNN "Voltage"
-F 5 "30%" H 5550 2750 60  0001 C CNN "Tolerance"
-F 6 "1276-2119-1-ND" H 5550 2750 60 0001 C CNN "Digi-Key Part Number"
-F 7 "CL10B822KB8NNNC" H 5550 2750 60 0001 C CNN "Manufacturer Part Number"
+F 5 "21%" H 5550 2750 60  0001 C CNN "Tolerance"
+F 6 "1276-1009-1-ND" H 5550 2750 60 0001 C CNN "Digi-Key Part Number"
+F 7 "CL10B103KB8NNNC" H 5550 2750 60 0001 C CNN "Manufacturer Part Number"
 F 8 "1.000000e-001" H 5550 2750 60 0001 C CNN "Price"
 	1    5550 2750
@@
 F 3 "http://www.samsungsem.com/servlet/FileDownload?type=spec&file=CL32B106KBJNFNE.pdf" H 5850 2750 60 0001 C CNN ""
 F 4 "50V" H 5850 2750 60  0001 C CNN "Voltage"
-F 5 "30%" H 5850 2750 60  0001 C CNN "Tolerance"
+F 5 "21%" H 5850 2750 60  0001 C CNN "Tolerance"
 F 6 "1276-3386-1-ND" H 5850 2750 60 0001 C CNN "Digi-Key Part Number"
 F 7 "CL32B106KBJNFNE" H 5850 2750 60 0001 C CNN "Manufacturer Part Number"
@@
 F 3 "http://www.samsungsem.com/servlet/FileDownload?type=spec&file=CL21B105KBFNNNE.pdf" H 3550 2950 60 0001 C CNN ""
 F 4 "50V" H 3550 2950 60  0001 C CNN "Voltage"
-F 5 "30%" H 3550 2950 60  0001 C CNN "Tolerance"
+F 5 "21%" H 3550 2950 60  0001 C CNN "Tolerance"
 F 6 "1276-1029-1-ND" H 3550 2950 60 0001 C CNN "Digi-Key Part Number"
 F 7 "CL21B105KBFNNNE" H 3550 2950 60 0001 C CNN "Manufacturer Part Number"
@@
 P 4650 1800
 F 0 "D1" H 4650 1900 50  0000 C CNN
-F 1 "TVS" H 4800 1700 40  0000 C CNN
+F 1 "TVScomA" H 4800 1700 40  0000 C CNN
 F 2 "~" H 4750 1800 60  0000 C CNN
 F 3 "http://www.littelfuse.com/~/media/electronics/datasheets/tvs_diode_arrays/littelfuse_tvs_diode_array_sm_datasheet.pdf.pdf" H 4750 1800 60 0001 C CNN ""
@@
 P 4650 2150
 F 0 "D2" H 4650 2250 50  0000 C CNN
-F 1 "TVS" H 4800 2050 40  0000 C CNN
+F 1 "TVScomA" H 4800 2050 40  0000 C CNN
 F 2 "~" H 4750 2150 60  0000 C CNN
 F 3 "http://www.littelfuse.com/~/media/electronics/datasheets/tvs_diode_arrays/littelfuse_tvs_diode_array_sm_datasheet.pdf.pdf" H 4750 2150 60 0001 C CNN ""
